File: unnamed.kicad_pcb (KiCad board)
At the start: 2 copper layers, 140 x 95 mm, 29 parts, among them J1 C128990, J2 C128990, SW1 KeySwitch, SW10 KeySwitch, SW11 KeySwitch, SW12 KeySwitch, SW13 KeySwitch, SW14 KeySwitch, SW15 KeySwitch, SW16 KeySwitch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

Commit message: update switch footprint, change 0805 to hand-solder footprint, update schematic value.
Parts:
- R1: footprint Resistor_SMD:R_0805_2012Metric -> Resistor_SMD:R_0805_2012Metric_Pad1.20x1.40mm_HandSolder
- R2: value 2.2K -> 1K; footprint Resistor_SMD:R_0805_2012Metric -> Resistor_SMD:R_0805_2012Metric_Pad1.20x1.40mm_HandSolder
- R3, R4: value 1K -> 100R; footprint Resistor_SMD:R_0805_2012Metric -> Resistor_SMD:R_0805_2012Metric_Pad1.20x1.40mm_HandSolder
- moved R2 1.00 mm to (203.2, 118.7)
- moved R4 0.30 mm to (202.5, 116.5)
Routing:
- net /SLIPT_HAND_PIN: track 55.2 -> 56.1 mm
- net /U0RX_: track 72.8 -> 73.4 mm
